File: HardWare/calculadora.kicad_sch (KiCad schematic)
At the start: 75 parts, among them J1 Screw_Terminal_01x02, J2 Screw_Terminal_01x02, J3 Screw_Terminal_01x02, J4 Screw_Terminal_01x02, J5 Conector ShiftRegister, J6 Screw_Terminal_01x14, Q1 Q_NPN_CBE, SW1 chave_tactil, SW10 chave_tactil, SW11 chave_tactil, SW12 chave_tactil, SW13 chave_tactil, SW14 chave_tactil, SW15 chave_tactil, SW16 chave_tactil, SW17 chave_tactil, SW18 chave_tactil, SW19 chave_tactil, SW2 chave_tactil, SW20 chave_tactil, SW21 chave_tactil, SW22 chave_tactil, SW23 chave_tactil, SW24 chave_tactil, SW25 chave_tactil, SW26 chave_tactil, SW27 chave_tactil, SW28 chave_tactil, SW29 chave_tactil, SW3 chave_tactil, SW30 chave_tactil, SW31 chave_tactil, SW32 chave_tactil, SW4 chave_tactil, SW5 chave_tactil, SW6 chave_tactil, SW7 chave_tactil, SW8 chave_tactil, SW9 chave_tactil, U1 ESP32-DEVKIT-V1, U2 LM358, U3 LM7805_TO220, U4 M74HC595B1, U5 LCD_GRAFICO_ST920

Commit message: Desenvolvido primeiro prototipo
Parts:
- removed C10, C11, C12: 0.1uf, Capacitor_THT:C_Disc_D7.5mm_W2.5mm_P5.00mm, symbol Device:C
- removed C2, C3, C4: 100UF/50v, Capacitor_THT:CP_Radial_D5.0mm_P2.50mm, symbol Device:C_Polarized
- removed C6, C7, C8: 10UF/35V, Capacitor_THT:CP_Radial_D5.0mm_P2.50mm, symbol Device:C_Polarized
- removed J2, J3, J4: Screw_Terminal_01x02, Connector_PinHeader_2.54mm:PinHeader_1x02_P2.54mm_Vertical, symbol Connector:Screw_Terminal_01x02
- removed J6: Screw_Terminal_01x14, Connector_PinHeader_2.54mm:PinHeader_1x14_P2.54mm_Horizontal, symbol Connector:Screw_Terminal_01x14
- added C2, C3: 0.1uf, Capacitor_THT:C_Disc_D7.5mm_W2.5mm_P5.00mm, symbol Device:C
- added D3: LED_IR, LED_THT:LED_D5.0mm, symbol Device:LED
- added Q2: Q_Photo_NPN, LED_THT:LED_D5.0mm, symbol Device:Q_Photo_NPN
- added R5, R6: 100, Resistor_THT:R_Axial_DIN0207_L6.3mm_D2.5mm_P10.16mm_Horizontal, symbol Device:R
- added R7: 100K, Resistor_THT:R_Axial_DIN0207_L6.3mm_D2.5mm_P10.16mm_Horizontal, symbol Device:R
- D2: value LED -> LED_RED
Connections:
- net +3V3: now also J5.2 (Pin_2), R7.2; no longer J5.1 (Pin_1)
- net +5V: now also RV2.3
- net GND: now also C18.2, C19.1, C20.2, C23.2, D2.1 (K), J5.3 (Pin_3), Q1.3 (E), R4.1, RV1.3, RV2.1, U1.2 (GND), U1.29 (GND), U4.13 (!G), U4.8 (GND), U5.1 (Vss), U5.20 (K(-)), C2.1, C3.1, D3.1 (K), Q2.2 (E)
- net GNDD: no longer C18.2, C19.1, C20.2, C23.2, J5.3 (Pin_3), Q1.3 (E), R4.1, RV1.3, U1.2 (GND), U1.29 (GND), U4.13 (!G), U4.8 (GND), U5.1 (Vss), U5.20 (K(-))
- net QH: now also J5.1 (Pin_1); no longer J5.2 (Pin_2)
- net Sinal_Analogico: now reaches RV2.2
- net Sinal_Analogico: now also U1.15 (D23), C3.2
- net at D2.2 (A): now also R6.2
- net Led_Ir: now reaches U1.10 (D19)
- net Led_Ir: now also R5.1
- net Led_Red: now reaches U1.11 (D21)
- net Led_Red: now also R6.1
- net Sensor_Ir: now reaches U1.14 (D22)
- net Sensor_Ir: now also C2.2, Q2.1 (C), R7.1
- new net: D3.2 (A), R5.2
Other:
- moved on the sheet: D2, RV2, U1
