File: HardWare/calculadora.kicad_pcb (KiCad board)
At the start: 2 copper layers, 100 x 150 mm, 75 parts, among them J1 Screw_Terminal_01x02, J2 Screw_Terminal_01x02, J3 Screw_Terminal_01x02, J4 Screw_Terminal_01x02, J5 Conector ShiftRegister, J6 Screw_Terminal_01x14, Q1 Q_NPN_CBE, SW1 chave_tactil, SW10 chave_tactil, SW11 chave_tactil, SW12 chave_tactil, SW13 chave_tactil, SW14 chave_tactil, SW15 chave_tactil, SW16 chave_tactil, SW17 chave_tactil, SW18 chave_tactil, SW19 chave_tactil, SW2 chave_tactil, SW20 chave_tactil, SW21 chave_tactil, SW22 chave_tactil, SW23 chave_tactil, SW24 chave_tactil, SW25 chave_tactil, SW26 chave_tactil, SW27 chave_tactil, SW28 chave_tactil, SW29 chave_tactil, SW3 chave_tactil, SW30 chave_tactil, SW31 chave_tactil, SW32 chave_tactil, SW4 chave_tactil, SW5 chave_tactil, SW6 chave_tactil, SW7 chave_tactil, SW8 chave_tactil, SW9 chave_tactil, U1 ESP32-DEVKIT-V1, U2 LM358, U3 LM7805_TO220, U4 M74HC595B1, U5 LCD_GRAFICO_ST920

Commit message: Desenvolvido primeiro prototipo
Parts:
- removed C10, C11, C12: 0.1uf, Capacitor_THT:C_Disc_D7.5mm_W2.5mm_P5.00mm
- removed C4: 100UF/50v, Capacitor_THT:CP_Radial_D5.0mm_P2.50mm
- removed C6, C7, C8: 10UF/35V, Capacitor_THT:CP_Radial_D5.0mm_P2.50mm
- removed J2, J3, J4: Screw_Terminal_01x02, Connector_PinHeader_2.54mm:PinHeader_1x02_P2.54mm_Vertical
- removed J6: Screw_Terminal_01x14, Connector_PinHeader_2.54mm:PinHeader_1x14_P2.54mm_Horizontal
- added D3: LED_IR, LED_THT:LED_D5.0mm, B.Cu at (102.2, 35.5)
- added Q2: Q_Photo_NPN, LED_THT:LED_D5.0mm, B.Cu at (121.7, 35.4)
- added R5: 100, Resistor_THT:R_Axial_DIN0207_L6.3mm_D2.5mm_P10.16mm_Horizontal, B.Cu at (105.2, 50.0)
- added R6: 100, Resistor_THT:R_Axial_DIN0207_L6.3mm_D2.5mm_P10.16mm_Horizontal, B.Cu at (113.4, 50.0)
- added R7: 100K, Resistor_THT:R_Axial_DIN0207_L6.3mm_D2.5mm_P10.16mm_Horizontal, B.Cu at (122.1, 39.8)
- C2, C3: value 100UF/50v -> 0.1uf; footprint Capacitor_THT:CP_Radial_D5.0mm_P2.50mm -> Capacitor_THT:C_Disc_D7.5mm_W2.5mm_P5.00mm
- D2: value LED -> LED_RED; moved to B.Cu
- RV2: moved to B.Cu
- moved C2 502.0 mm to (118.7, 45.2), turned to 90 degrees
- moved C3 490.2 mm to (132.6, 51.8), turned to 180 degrees
- moved C24 476.8 mm to (104.0, 68.4), turned to 90 degrees
- moved C25 468.1 mm to (109.7, 68.4), turned to 90 degrees
- moved C19 372.8 mm to (91.0, 72.7), turned to -90 degrees
- moved C20 371.0 mm to (88.0, 77.7), turned to 180 degrees
- moved BZ1 368.0 mm to (129.6, 74.0)
- moved C1 368.0 mm to (47.9, 38.9)
- moved C13 368.0 mm to (43.8, 43.6)
- moved C14 368.0 mm to (39.4, 47.0)
- moved C15 368.0 mm to (126.6, 106.5)
- moved C5 368.0 mm to (53.1, 38.8)
- moved C9 368.0 mm to (57.1, 43.6)
- moved D1 368.0 mm to (39.4, 60.3)
- moved J1 368.0 mm to (51.7, 34.2)
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Connections:
- C2 pad 1: VCC -> GNDD
- C2 pad 2: GND -> Sensor_Ir
- C3 pad 1: +5V -> GNDD
- C3 pad 2: GND -> Sinal_Analogico
- D2 pad 1: unconnected-(D2-Pad1) -> GNDD
- D2 pad 2: unconnected-(D2-Pad2) -> Net-(D2-Pad2)
- J5 pad 1: +3V3 -> QH
- J5 pad 2: QH -> +3V3
- RV2 pad 1: unconnected-(RV2-Pad1) -> GNDD
- RV2 pad 2: unconnected-(RV2-Pad2) -> Sinal_Analogico
- RV2 pad 3: unconnected-(RV2-Pad3) -> +5V
- U1 pad 10: unconnected-(U1-Pad10) -> Led_Ir
- U1 pad 11: unconnected-(U1-Pad11) -> Led_Red
- U1 pad 14: unconnected-(U1-Pad14) -> Sensor_Ir
- U1 pad 15: unconnected-(U1-Pad15) -> Sinal_Analogico
Routing:
- net QH: track 0.00 -> 72.6 mm
- net +3V3: track 97.7 -> 157.4 mm
- net CLOCK_SHIFT: track 48.3 -> 95.6 mm
- net SET_SHIFT: track 44.4 -> 91.4 mm
- net +5V: vias 0 -> 2

Commit message: Ajustes
Parts:
- moved C3 1.48 mm to (131.1, 51.9)
- moved RV2 0.32 mm to (132.2, 47.8)
Connections:
- C18 pad 2: GNDD -> GND
- C19 pad 1: GNDD -> GND
- C2 pad 1: GNDD -> GND
- C20 pad 2: GNDD -> GND
- C23 pad 2: GNDD -> GND
- C3 pad 1: GNDD -> GND
- D2 pad 1: GNDD -> GND
- D3 pad 1: GNDD -> GND
- J5 pad 3: GNDD -> GND
- Q1 pad 3: GNDD -> GND
- Q2 pad 2: GNDD -> GND
- R4 pad 1: GNDD -> GND
- RV1 pad 3: GNDD -> GND
- RV2 pad 1: GNDD -> GND
- U1 pad 2: GNDD -> GND
- U1 pad 29: GNDD -> GND
- U4 pad 13: GNDD -> GND
- U4 pad 8: GNDD -> GND
- U5 pad 1: GNDD -> GND
- U5 pad 20: GNDD -> GND
Routing:
- net Sensor_Ir: track 0.00 -> 85.3 mm
- net Sinal_Analogico: track 0.00 -> 79.4 mm
- net Led_Red: track 0.00 -> 71.1 mm
- net Led_Ir: track 0.00 -> 66.0 mm
- net +3V3: track 157.4 -> 218.1 mm
- net +5V: track 215.6 -> 267.8 mm
- net Net-(D3-Pad2): track 0.00 -> 4.62 mm
- net Net-(D2-Pad2): track 0.00 -> 4.61 mm
- added copper zone on B.Cu, net GND
